File: docs/aqua_pcb_schem/aqua_pcb_schem.kicad_sch (KiCad schematic)
At the start: 35 parts, among them J1 Connector, J2 Vin_5V, J3 pH Probe, Q1 SS8050, Q2 SS8050, SW1 SW_Push, SW2 SW_Push, U1 TLC4502, U3 DS18B20, U4 AZ1117-3.3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

Commit message: schematic and parts all finalized. gotta order today
Parts:
- removed J2: Vin_5V, symbol Connector_Generic:Conn_01x01
- removed U1, U7: TLC4502, symbol Amplifier_Operational:LM358
- removed U3: DS18B20, Package_TO_SOT_THT:TO-92_Inline, symbol Sensor_Temperature:DS18B20
- added C10: 100 [uF], Capacitor_SMD:C_0805_2012Metric_Pad1.18x1.45mm_HandSolder, symbol Device:C
- added C8: 0.1 [uF], Capacitor_SMD:C_0805_2012Metric_Pad1.18x1.45mm_HandSolder, symbol Device:C
- added C9: 10 [uF], Capacitor_SMD:C_0805_2012Metric_Pad1.18x1.45mm_HandSolder, symbol Device:C
- added H1, H2, H3, H4: MountingHole, MountingHole:MountingHole_3.2mm_M3, symbol Mechanical:MountingHole
- added J4: USB-UART Header, Package_DFN_QFN:QFN-64-1EP_9x9mm_P0.5mm_EP4.1x4.1mm, symbol Connector_Generic:Conn_01x05
- added J5: USB_C_Receptacle_PowerOnly_6P, Connector_USB:USB_C_Receptacle_Amphenol_124019772112A, symbol Connector:USB_C_Receptacle_PowerOnly_6P
- added U1, U2: TLC4502, Package_TO_SOT_SMD:SOT-353_SC-70-5, symbol Amplifier_Operational:TLV172IDCK
- C1, C4, C5, C6, C7: footprint (none) -> Capacitor_SMD:C_0805_2012Metric_Pad1.18x1.45mm_HandSolder
- C2, C3: value 0.1 [uF] -> 10 [uF]; footprint (none) -> Capacitor_SMD:C_0805_2012Metric_Pad1.18x1.45mm_HandSolder
- J1: value Connector -> DS18B20; footprint (none) -> TerminalBlock_Phoenix:TerminalBlock_Phoenix_PT-1,5-2-3.5-H_1x02_P3.50mm_Horizontal
- J3: footprint (none) -> Connector_Coaxial:BNC_Amphenol_031-6575_Horizontal
- JP1: footprint (none) -> Jumper:SolderJumper-3_P1.3mm_Open_Pad1.0x1.5mm
- R1, R10, R11, R12, R13, R14, R15, R2, R4, R5, R6, R8, R9: footprint (none) -> Resistor_SMD:R_0805_2012Metric_Pad1.20x1.40mm_HandSolder
- R3: value 30 [kΩ] -> 10 [kΩ]; footprint (none) -> Resistor_SMD:R_0805_2012Metric_Pad1.20x1.40mm_HandSolder
- SW1, SW2: footprint (none) -> Button_Switch_THT:SW_PUSH_1P1T_6x3.5mm_H5.0_APEM_MJTP1250
- U4: footprint (none) -> Package_TO_SOT_SMD:SOT-223
Connections:
- net +3.3 [V]: now also U1.5 (V+), U2.5 (V+); no longer C2.1, C3.1
- net GND: now also C10.2, C8.2, C9.2, J4.5 (Pin_5), J5.A12 (GND), J5.B12 (GND), U1.2 (V-), U2.2 (V-)
- net RTS: now reaches Q1.2 (E), R14.1
- net RTS: now also J4.1 (Pin_1)
- net at C7.1, R5.2, R6.1: now also U1.1 (+)
- net GPIO46_Strapping: now reaches R8.1
- net GPIO46_Strapping: now also U6.16 (IO46)
- net temp: now reaches J1.1 (Pin_1), R1.1
- net temp: now also U6.4 (IO4)
- net GPIO0_Strapping: now reaches R13.2
- net GPIO0_Strapping: now also C5.1, R10.1, SW1.2, U6.27 (IO0)
- net CHIP_PU: now reaches R12.2
- net CHIP_PU: now also C6.1, R11.1, SW2.2, U6.3 (EN)
- net pH: now reaches R3.1
- net pH: now also U6.5 (IO5), U2.4
- net at R2.2, R3.2: now also U2.3 (-)
- net GPIO3_Strapping: now reaches R9.1
- net GPIO3_Strapping: now also U6.15 (IO3)
- net +3.3 V: now reaches U4.2 (VO), U6.2 (3V3)
- net +3.3 V: now also C3.1, C10.1, C8.1, C9.1
- net RXD: now reaches U6.36 (RXD0)
- net RXD: now also J4.4 (Pin_4)
- net TXD: now reaches U6.37 (TXD0)
- net TXD: now also J4.3 (Pin_3)
- net DTR: now reaches Q2.3 (C), R15.1
- net DTR: now also J4.2 (Pin_2)
- net electrode +: now reaches J3.1 (Pin_1)
- net electrode +: now also U2.1 (+)
- net electrode -: now reaches J3.2 (Pin_2)
- net electrode -: now also U1.3 (-), U1.4
- net +5 [V] renamed +5 V
- net +5 V: now also C2.1, J5.A9 (VBUS), J5.B9 (VBUS)
Other:
- note added: "(5) Wall Step-Down"
- note removed: "(5) Decoupling Capacitors"
- note removed: "+5 [V]"
- note removed: "CHIP_PU"
- note removed: "DTR"
- note removed: "GPIO0_Strapping"
- note removed: "GPIO3_Strapping"
- note removed: "GPIO46_Strapping"
- note removed: "RTS"
- note removed: "electrode +"
- note removed: "electrode -"
- note removed: "pH"
- note removed: "temp"
- moved on the sheet: C1, C2, C3, C5, C6, J1, JP1, Q1, Q2, R1, R10, R11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
